File: V-00684-00.brd (EAGLE design)
At the start: 162 x 102 mm, 11 parts, among them J11 22-05-7028-02, J12 22-05-7028-02, J13 22-05-7028-02, J5 22-05-7048-04, J8 22-05-7048-04, J9 22-05-7048-04

Commit message: Save
Parts:
- J11: value 22-05-7028-02 -> MOTOR4_Ref
- J12: value 22-05-7028-02 -> MOTOR5_Ref
- J13: value 22-05-7028-02 -> MOTOR6_Ref
- J5: value 22-05-7048-04 -> MOTOR4
- J8: value 22-05-7048-04 -> MOTOR5
- J9: value 22-05-7048-04 -> MOTOR6
- moved J13 58.1 mm to (44.0, 15.0), turned to 90 degrees
- moved J11 49.6 mm to (44.0, -15.0), turned to 90 degrees
- moved J12 49.6 mm to (44.0, 0.00), turned to 90 degrees
- moved J9 5.94 mm to (106.0, -15.0)
- moved J8 4.63 mm to (106.0, 0.00)
- moved R4 3.81 mm to (9.99, 30.4), turned to 180 degrees
- moved R1 3.71 mm to (10.0, 38.3)
- moved J5 3.30 mm to (106.0, 15.0)
Connections:
- net M4A1 renamed N.C.0
- net M4A2 renamed N.C.1
- net M4B1 renamed N.C.2
- net M4B2 renamed N.C.3
- removed net M1A2: J1.C8
- removed net M1B2: J1.C10
- removed net M1_REF_L: J1.C24
- removed net M2A2: J1.C12
- removed net M2B2: J1.C14
- removed net M2_REF_L: J1.A26
- removed net M3A2: J1.C16
- removed net M3B2: J1.C18
- removed net M3_REF_L: J1.C26
- removed net M4_REF_L: J1.A28
- removed net N$10: J5.4
- removed net N$11: J5.3
- removed net N$12: J5.2
- removed net N$13: J5.1
- removed net N$14: J8.4
- removed net N$15: J8.3
- removed net N$16: J8.2
- removed net N$17: J8.1
- removed net N$18: J9.4
- removed net N$19: J9.3
- removed net N$2: J11.2
- removed net N$20: J9.2
- removed net N$21: J9.1
- removed net N$4: J11.1
- removed net N$5: J13.2
- removed net N$7: J13.1
- removed net N$8: J12.2
- removed net N$9: J12.1
- new net !M1A1: J1.C8, J5.3
- new net !M1B1: J1.C10, J5.1
- new net !M2A1: J1.C12, J8.3
- new net !M2B1: J1.C14, J8.1
- new net !M3A1: J1.C16, J9.3
- new net !M3B1: J1.C18, J9.1
- new net M1_REF: J1.A24, J11.2
- new net M2_REF: J1.A26, J12.2
- new net M3_REF: J1.A28, J13.2
- net GND: now also J1.C24, J1.C26, J11.1, J12.1, J13.1; no longer J1.A24
- net M1A1: now also J5.4
- net M1B1: now also J5.2
- net M2A1: now also J8.4
- net M2B1: now also J8.2
- net M3A1: now also J9.4
- net M3B1: now also J9.2
Routing:
- net M3_REF: track 0.00 -> 193.9 mm
- net M2_REF: track 0.00 -> 173.8 mm
- net M1_REF: track 0.00 -> 151.5 mm
- net +24V: track 0.00 -> 145.2 mm
- net +5V: track 0.00 -> 140.9 mm
- net M3A1: track 2.93 -> 56.0 mm
- net M3B1: track 2.93 -> 55.9 mm
- net M2B1: track 2.93 -> 54.0 mm
- net M2A1: track 2.93 -> 53.9 mm
- net !M3A1: track 0.00 -> 49.8 mm
- net !M3B1: track 0.00 -> 49.8 mm
- net M1A1: track 2.93 -> 51.9 mm
- net M1B1: track 2.93 -> 51.9 mm
- net !M2B1: track 0.00 -> 47.8 mm
- net !M2A1: track 0.00 -> 47.8 mm
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Other:
- board text added: "V-00684-00 LIC_rack_BM4_Focus-00 Lukas Novak 13.11.2015"
- board text removed: "V-00684-00 LIC_rack_BM4_Focus-00 Lukas Novak 06.11.2015"
