File: V-00684-00.sch (EAGLE design)
At the start: 11 parts, among them J11 22-05-7028-02, J12 22-05-7028-02, J13 22-05-7028-02, J5 22-05-7048-04, J8 22-05-7048-04, J9 22-05-7048-04

Commit message: Save
Parts:
- J11: value 22-05-7028-02 -> MOTOR4_Ref
- J12: value 22-05-7028-02 -> MOTOR5_Ref
- J13: value 22-05-7028-02 -> MOTOR6_Ref
- J5: value 22-05-7048-04 -> MOTOR4
- J8: value 22-05-7048-04 -> MOTOR5
- J9: value 22-05-7048-04 -> MOTOR6
Connections:
- net M4A1 renamed N.C.0
- net M4A2 renamed N.C.1
- net M4B1 renamed N.C.2
- net M4B2 renamed N.C.3
- removed net M1A2: J1-C8.MS
- removed net M1B2: J1-C10.MS
- removed net M1_REF_L: J1-C24.MS
- removed net M2A2: J1-C12.MS
- removed net M2B2: J1-C14.MS
- removed net M2_REF_L: J1-A26.MS
- removed net M3A2: J1-C16.MS
- removed net M3B2: J1-C18.MS
- removed net M3_REF_L: J1-C26.MS
- removed net M4_REF_L: J1-A28.MS
- removed net N$10: J5-4.S
- removed net N$11: J5-3.S
- removed net N$12: J5-2.S
- removed net N$13: J5-1.S
- removed net N$14: J8-4.S
- removed net N$15: J8-3.S
- removed net N$16: J8-2.S
- removed net N$17: J8-1.S
- removed net N$18: J9-4.S
- removed net N$19: J9-3.S
- removed net N$2: J11-2.S
- removed net N$20: J9-2.S
- removed net N$21: J9-1.S
- removed net N$4: J11-1.S
- removed net N$5: J13-2.S
- removed net N$7: J13-1.S
- removed net N$8: J12-2.S
- removed net N$9: J12-1.S
- new net !M1A1: J1-C8.MS, J5-3.S
- new net !M1B1: J1-C10.MS, J5-1.S
- new net !M2A1: J1-C12.MS, J8-3.S
- new net !M2B1: J1-C14.MS, J8-1.S
- new net !M3A1: J1-C16.MS, J9-3.S
- new net !M3B1: J1-C18.MS, J9-1.S
- new net M1_REF: J1-A24.MS, J11-2.S
- new net M2_REF: J1-A26.MS, J12-2.S
- new net M3_REF: J1-A28.MS, J13-2.S
- net GND: now also J1-C24.MS, J1-C26.MS, J11-1.S, J12-1.S, J13-1.S; no longer J1-A24.MS
- net M1A1: now also J5-4.S
- net M1B1: now also J5-2.S
- net M2A1: now also J8-4.S
- net M2B1: now also J8-2.S
- net M3A1: now also J9-4.S
- net M3B1: now also J9-2.S
